File: kicad_schema_emitter/rc-emitter_tft_trim_board.sch (KiCad schematic (older format))
At the start: 5 parts, among them J2 JST_cable, SW2 SW_Push, SW4 SW_Push

Commit message: Update
Parts:
- J2: footprint Connector_PinHeader_2.54mm:PinHeader_1x03_P2.54mm_Vertical -> Connector_JST:JST_XH_B3B-XH-A_1x03_P2.50mm_Vertical
- renumbered R2 to R1, R4 to R2, SW2 to SW1, SW4 to SW2
Other:
- note added: "!! Last module R2 = 2K !!"
- note added: "5V"
- note added: "6 items"
- note added: "In"
- note added: "Out\n"
- note removed: "4 items"
Changed lines of the file:
@@
 $EndDescr
 $Comp
-L Switch:SW_Push SW2
+L Switch:SW_Push SW1
 U 1 1 5F524B50
 P 4850 5150
-F 0 "SW2" H 4850 5435 50  0000 C CNN
+F 0 "SW1" H 4850 5435 50  0000 C CNN
 F 1 "SW_Push" H 4850 5344 50  0000 C CNN
 F 2 "Button_Switch_THT:SW_PUSH_6mm_H4.3mm" H 4850 5350 50  0001 C CNN
@@
 $EndComp
 $Comp
-L Switch:SW_Push SW4
+L Switch:SW_Push SW2
 U 1 1 5F524B56
 P 5350 5150
-F 0 "SW4" H 5350 5435 50  0000 C CNN
+F 0 "SW2" H 5350 5435 50  0000 C CNN
 F 1 "SW_Push" H 5350 5344 50  0000 C CNN
 F 2 "Button_Switch_THT:SW_PUSH_6mm_H4.3mm" H 5350 5350 50  0001 C CNN
@@
 F 0 "J2" H 6230 5542 50  0000 L CNN
 F 1 "JST_cable" H 6230 5451 50  0000 L CNN
-F 2 "Connector_PinHeader_2.54mm:PinHeader_1x03_P2.54mm_Vertical" H 6150 5500 50  0001 C CNN
+F 2 "Connector_JST:JST_XH_B3B-XH-A_1x03_P2.50mm_Vertical" H 6150 5500 50  0001 C CNN
 F 3 "~" H 6150 5500 50  0001 C CNN
 	1    6150 5500
@@
 	5350 4500 5550 4500
 $Comp
-L Device:R R4
+L Device:R R2
 U 1 1 5F524B62
 P 5700 4500
-F 0 "R4" H 5630 4454 50  0000 R CNN
+F 0 "R2" H 5630 4454 50  0000 R CNN
 F 1 "220ohm" H 5630 4545 50  0000 R CNN
 F 2 "Resistor_THT:R_Axial_DIN0207_L6.3mm_D2.5mm_P10.16mm_Horizontal" V 5630 4500 50  0001 C CNN
@@
 $EndComp
 $Comp
-L Device:R R2
+L Device:R R1
 U 1 1 5F524B5C
 P 5200 4500
-F 0 "R2" H 5130 4454 50  0000 R CNN
+F 0 "R1" H 5130 4454 50  0000 R CNN
 F 1 "220ohm" H 5130 4545 50  0000 R CNN
 F 2 "Resistor_THT:R_Axial_DIN0207_L6.3mm_D2.5mm_P10.16mm_Horizontal" V 5130 4500 50  0001 C CNN
@@
 Connection ~ 5050 4500
 Text Notes 4800 4350 0    50   ~ 0
-4 items
+6 items
 Wire Notes Line
 	4500 4400 6650 4400
@@
 Wire Notes Line
 	4500 5950 4500 4400
+Text Notes 5500 4350 0    50   ~ 0
+!! Last module R2 = 2K !!
+Text Notes 5750 5850 0    50   ~ 0
+5V
+Text Notes 5850 5000 0    50   ~ 0
+Out\n
+Text Notes 5700 5500 0    50   ~ 0
+In
 $EndSCHEMATC
