File: kicad_schema_emitter/rc-emitter_tft.kicad_pcb (KiCad board)
At the start: 2 copper layers, 23 parts, among them J1 nrf24L01+PA+lna, J2 Conn_01x03, J3 Conn_01x03, J4 Conn_01x03, J5 Conn_01x03, J6 menu + OK, J7 left + right, J8 Gim_left, J9 Gim_right, U0 ATmega328P-PU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

Commit message: Files Selection git
Parts:
- added J10: Conn_01x05, Connector_PinHeader_2.54mm:PinHeader_1x05_P2.54mm_Vertical, F.Cu at (120.7, 71.1)
- J2: value Conn_01x03 -> roll_trim
- J3: value Conn_01x03 -> pitch_trim
- J4: value Conn_01x03 -> yaw_trim
- J5: value Conn_01x03 -> throttle_trim
- J6: value menu + OK -> menu_ok_back
- J7: value left + right -> menu_nav
- R1: renamed from R1 510Ω
- R14: value 10KΩ -> 10Kohm
- R2: renamed from R2 330Ω
- R3: value 220Ω -> 220ohm
- RV1: footprint potentiometer_WHT148:WH148 -> Connector_PinHeader_2.54mm:PinHeader_1x03_P2.54mm_Vertical
- moved C4 99.7 mm to (86.4, 50.8)
- moved 100nF1 93.3 mm to (88.7, 46.3)
- moved R1 93.3 mm to (101.7, 45.3)
- moved R2 93.3 mm to (96.7, 45.3)
- moved C2 92.6 mm to (99.3, 59.7)
- moved RV1 92.5 mm to (81.3, 67.3)
- moved U1 89.9 mm to (88.9, 58.4)
- moved J9 81.3 mm to (110.5, 45.7)
- moved J5 72.0 mm to (127.0, 66.0), turned to 0 degrees
- moved J4 65.1 mm to (127.0, 55.9), turned to 0 degrees
- moved J1 63.4 mm to (110.5, 33.0), turned to 90 degrees
- moved J2 51.7 mm to (127.0, 35.6), turned to 0 degrees
- moved LCD1 47.2 mm to (119.4, 91.4)
- moved R3 45.6 mm to (96.5, 96.5)
- moved C1 41.7 mm to (87.6, 73.7), turned to 90 degrees
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- renumbered .1 to LCD1
Connections:
- J1 pad 8: (no net) -> Net-(J1-Pad8)
- J2 pad 2: (no net) -> Net-(J2-Pad2)
- LCD1 pad 10: (no net) -> Net-(LCD1-Pad10)
- LCD1 pad 5: Net-(.1-Pad5) -> GND
- LCD1 pad 6: GND -> Net-(LCD1-Pad6)
- LCD1 pad 7: (no net) -> Net-(LCD1-Pad7)
- LCD1 pad 8: (no net) -> Net-(LCD1-Pad8)
- LCD1 pad 9: (no net) -> Net-(LCD1-Pad9)
- RV1 pad 1: GND -> +5V
- U0 pad 1: (no net) -> Net-(J10-Pad2)
- U0 pad 2: (no net) -> Net-(J10-Pad3)
- U0 pad 20: (no net) -> Net-(U0-Pad20)
- U0 pad 21: (no net) -> Net-(U0-Pad21)
- U0 pad 28: (no net) -> Net-(J10-Pad1)
- U0 pad 3: (no net) -> Net-(J10-Pad4)
- U0 pad 4: (no net) -> Net-(J10-Pad5)
- U0 pad 6: Net-(.1-Pad5) -> Net-(LCD1-Pad6)
Routing:
- net +5V: track 0.00 -> 182.5 mm
- net GND: track 0.00 -> 143.0 mm
- net Net-(J1-Pad4): track 0.00 -> 74.8 mm
- net Net-(J1-Pad7): track 0.00 -> 70.1 mm
- net Net-(J1-Pad6): track 0.00 -> 66.9 mm
- net Net-(J1-Pad3): track 0.00 -> 65.4 mm
- net Net-(J1-Pad5): track 0.00 -> 63.0 mm
- net 3.2V: track 0.00 -> 58.7 mm
- net Net-(J9-Pad4): track 0.00 -> 45.8 mm
- net Net-(J9-Pad3): track 0.00 -> 45.1 mm
- net Net-(LCD1-Pad3): track 0.00 -> 44.9 mm
- net Net-(J8-Pad3): track 0.00 -> 35.9 mm
- net Net-(J8-Pad4): track 0.00 -> 32.8 mm
- net Net-(J7-Pad1): track 0.00 -> 23.0 mm
- net Net-(R1-Pad1): track 0.00 -> 22.1 mm
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Other:
- board outline added: 61 x 77.5 mm
- board text added: "By: 2CoB9 https://github.com/CoMeister/"
- board text added: "GND"
- board text added: "GNU GPL V3 29.06.2007"
- board text added: "IN"
- board text added: "JLCJLCJLCJLC"
- board text added: "MegaRC"
- board text added: "OUT"
- board text added: "PC5/A5"
- board text added: "PC6/RESET"
- board text added: "PD0/0_RX"
- board text added: "PD1/1_TX"
- board text added: "PD2/2"
- board text added: "VCC"
- board text removed: "<35mm from bottom to first pins nRF24L01"
