File: kicad_schema_emitter/rc-emitter_tft.sch (KiCad schematic (older format))
At the start: 25 parts, among them J1 nrf24L01+PA+lna, J2 Conn_01x03, J3 Conn_01x03, J4 Conn_01x03, J5 Conn_01x03, SW10 SW_Push_up, SW11 SW_Push_down, SW12 SW_Push_ok/modify, SW9 SW_Push_Menu/back, U0 ATmega328P-PU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

Commit message: Update
Parts:
- removed R11, R12, R13: 220ohm, Resistor_THT:R_Axial_DIN0207_L6.3mm_D2.5mm_P10.16mm_Horizontal, symbol Device:R
- removed R15: 2Kohm, Resistor_THT:R_Axial_DIN0207_L6.3mm_D2.5mm_P10.16mm_Horizontal, symbol Device:R
- removed SW10: SW_Push_up, Button_Switch_THT:SW_PUSH_6mm_H4.3mm, symbol Switch:SW_Push
- removed SW11: SW_Push_down, Button_Switch_THT:SW_PUSH_6mm_H4.3mm, symbol Switch:SW_Push
- removed SW12: SW_Push_ok/modify, Button_Switch_THT:SW_PUSH_6mm_H4.3mm, symbol Switch:SW_Push
- removed SW9: SW_Push_Menu/back, Button_Switch_THT:SW_PUSH_6mm_H4.3mm, symbol Switch:SW_Push
- removed screen1: ST7735, Connector_PinHeader_2.54mm:PinHeader_1x08_P2.54mm_Vertical, symbol Display_Graphipersoc:ST7735
- added .1: BTC-2004B, Connector_PinHeader_2.54mm:PinHeader_1x16_P2.54mm_Vertical, symbol lcd2004:BTC-2004B
- added J6: menu + OK, Connector_JST:JST_XH_B3B-XH-A_1x03_P2.50mm_Vertical, symbol Connector_Generic:Conn_01x03
- added J7: left + right, Connector_JST:JST_XH_B3B-XH-A_1x03_P2.50mm_Vertical, symbol Connector_Generic:Conn_01x03
- added J8: Gim_left, Connector_JST:JST_XH_B4B-XH-A_1x04_P2.50mm_Vertical, symbol Connector_Generic:Conn_01x04
- added J9: Gim_right, Connector_JST:JST_XH_B4B-XH-A_1x04_P2.50mm_Vertical, symbol Connector_Generic:Conn_01x04
- added R3: 220ohm, Resistor_THT:R_Axial_DIN0207_L6.3mm_D2.5mm_P10.16mm_Horizontal, symbol Device:R
- added RV1: R_POT, potentiometer_WHT148:WH148, symbol Device:R_POT
- J1: symbol Connector_Generic:Conn_02x04_Top_Bottom -> Connector_Generic:Conn_02x04_Odd_Even
Connections:
- net +5V: now also U1.3 (VI), .1.2 (VCC), J6.3 (Pin_3), J7.3 (Pin_3), J8.2 (Pin_2), J9.2 (Pin_2), R3.2; no longer U1.2 (VO)
- net 3.2V: now also J1.2 (Pin_2), U1.2 (VO); no longer J1.5 (Pin_5), U1.1 (ADJ)
- net GND: now also .1.1 (GND), .1.16 (K), .1.6 (RW), J8.1 (Pin_1), J9.1 (Pin_1), RV1.1, RV1.3
- net at U0.11 (PD5): now also .1.11 (D4)
- net at U0.12 (PD6): now also .1.12 (D5)
- net at U0.13 (PD7): now also .1.13 (D6)
- net at U0.14 (PB0): now also .1.14 (D7)
- net at U0.15 (PB1): now also J1.3 (Pin_3); no longer J1.2 (Pin_2)
- net at U0.16 (PB2): now also J1.4 (Pin_4); no longer J1.6 (Pin_6)
- net at U0.17 (PB3): now also J1.6 (Pin_6); no longer J1.7 (Pin_7)
- net at U0.18 (PB4): now also J1.7 (Pin_7); no longer J1.4 (Pin_4)
- net at U0.19 (PB5): now also J1.5 (Pin_5); no longer J1.3 (Pin_3)
- net at U0.23 (PC0): now also J9.3 (Pin_3)
- net at U0.24 (PC1): now also J9.4 (Pin_4)
- net at U0.25 (PC2): now also J8.3 (Pin_3)
- net at U0.26 (PC3): now also J8.4 (Pin_4)
- net at R14.1, U0.27 (PC4): now also J7.1 (Pin_1)
- net at U0.5 (PD3): now also .1.4 (RS)
- net at U0.6 (PD4): now also .1.5 (EN)
- net at J5.1 (Pin_1): now also J6.2 (Pin_2)
- net at R1.1, R2.1: now also U1.1 (ADJ); no longer U1.3 (VI)
- new net: .1.15 (A), R3.1
- new net: .1.3 (VC), RV1.2
- new net: J6.1 (Pin_1), J7.2 (Pin_2)
- no-connect marks 21 -> 13
Other:
- note added: "5V to 3.2V for \nnRF24L01+"
- note removed: "5V to 3.2V for \nnRF24L01+ and \nLED of ST7735"
- moved on the sheet: 100nF1, C0, C1, C2, R1, R14, R2, U1, Y1

Commit message: Files Selection git
Parts:
- added J10: Conn_01x05, Connector_PinHeader_2.54mm:PinHeader_1x05_P2.54mm_Vertical, symbol Connector_Generic:Conn_01x05
- J2: value Conn_01x03 -> roll_trim
- J3: value Conn_01x03 -> pitch_trim
- J4: value Conn_01x03 -> yaw_trim
- J5: value Conn_01x03 -> throttle_trim
- J6: value menu + OK -> menu_ok_back
- J7: value left + right -> menu_nav
- LCD1: renamed from .1; symbol lcd2004:BTC-2004B -> rc-emitter_tft-rescue:BTC-2004B-lcd2004
- RV1: footprint potentiometer_WHT148:WH148 -> Connector_PinHeader_2.54mm:PinHeader_1x03_P2.54mm_Vertical
Connections:
- net +5V: now also RV1.1
- net GND: now also LCD1.5 (RW); no longer LCD1.6 (RW), RV1.1
- net at U0.1 (~RESET~/PC6): now also J10.2 (Pin_2)
- net at U0.2 (PD0): now also J10.3 (Pin_3)
- net at U0.28 (PC5): now also J10.1 (Pin_1)
- net at U0.3 (PD1): now also J10.4 (Pin_4)
- net at U0.4 (PD2): now also J10.5 (Pin_5)
- net at U0.6 (PD4): now also LCD1.6 (EN); no longer LCD1.5 (EN)
- no-connect marks 13 -> 8
Other:
- moved on the sheet: J2, J3, J4, J5, J6, J7, J8, R14
