File: kicad_schema_emitter/rc-emitter_tft_trim_board.kicad_pcb (KiCad board)
At the start: 2 copper layers, 14 x 46 mm, 7 parts, among them J2 JST_cable, SW2 SW_Push, SW4 SW_Push

Commit message: Update
Parts:
- removed REF** (x2): MountingHole_3.2mm_M3, MountingHole:MountingHole_3.2mm_M3
- renumbered R2 to R1, R4 to R2, SW2 to SW1, SW4 to SW2
Other:
- outline, holes or cut-outs redrawn

Commit message: Files Selection git
Parts:
- R1 220ohm: renamed from R1
Routing:
- net Net-(R1-Pad2): track 13.4 -> 30.1 mm
- net Net-(J2-Pad1): track 4.50 -> 5.62 mm
- net Net-(J2-Pad2): track 32.8 -> 32.3 mm
Other:
- board size 14 x 46 mm -> 14 x 53.3 mm
- board text added: "By: 2CoB9 https://github.com/CoMeister/"
- board text added: "GNU GPL V3 29.06.2007"
- board text added: "IN"
- board text added: "JLCJLCJLCJLC"
- board text added: "MegaRC"
- board text added: "OUT"
- board text added: "VCC"
